File: iPot/iPot-cb.sch (KiCad schematic (older format))
At the start: 43 parts, among them CON1 12VDC, IC1 ATMEGA644-P, P1 JTAG, P10 SPRAY_PUMP, P11 USB_PWR, P2 SPI, P3 UART, P4 SOIL, P5 TEMP/HUMID, P6 LIGHT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

Commit message: Little bit of general purpose design
Parts:
- added D10, D3, D4, D5, D6, D7, D8, D9: 1N4148, Diodes_ThroughHole:Diode_DO-35_SOD27_Horizontal_RM10, symbol D
- added IC2: L298, TO_SOT_Packages_THT:Multiwatt_15_Vertical, symbol L298
- added P11: I2C4, Pin_Headers:Pin_Header_Straight_1x04, symbol CONN_01X04
- added P13: USB_PWR2, Connect:USB_A_Vertical, symbol USB_A
- C2: renamed from C5; footprint (none) -> Capacitors_ThroughHole:C_Disc_D6_P5
- C3: renamed from C6; footprint (none) -> Capacitors_ThroughHole:C_Disc_D3_P2.5
- C4: renamed from C3; footprint (none) -> Capacitors_ThroughHole:C_Disc_D6_P5
- C5: renamed from C1; footprint (none) -> Capacitors_ThroughHole:C_Disc_D3_P2.5
- C6: renamed from C2; footprint (none) -> Capacitors_ThroughHole:C_Disc_D3_P2.5
- P1: renamed from P9; footprint (none) -> Terminal_Blocks:TerminalBlock_Pheonix_MKDS1.5-2pol
- P10: renamed from P6; value LIGHT -> I2C3; footprint (none) -> Pin_Headers:Pin_Header_Straight_1x04
- P2: renamed from P10; footprint (none) -> Terminal_Blocks:TerminalBlock_Pheonix_MKDS1.5-2pol
- P5: renamed from P11; value USB_PWR -> USB_PWR1; footprint Connect:USB_A -> Connect:USB_A_Vertical
- P8: renamed from P4; value SOIL -> I2C1; footprint (none) -> Pin_Headers:Pin_Header_Straight_1x04
- P9: renamed from P5; value TEMP/HUMID -> I2C2; footprint (none) -> Pin_Headers:Pin_Header_Straight_1x04
- Q1: renamed from Q5; footprint (none) -> TO_SOT_Packages_THT:TO-92_Inline_Wide
- Q2: renamed from Q1; footprint (none) -> TO_SOT_Packages_THT:TO-220_Neutral123_Vertical
- Q3: renamed from Q2; footprint (none) -> TO_SOT_Packages_THT:TO-220_Neutral123_Vertical
- Q4: renamed from Q3; footprint (none) -> TO_SOT_Packages_THT:TO-92_Inline_Wide
- Q5: renamed from Q4; footprint (none) -> TO_SOT_Packages_THT:TO-92_Inline_Wide
- Q6: footprint (none) -> TO_SOT_Packages_THT:TO-92_Inline_Wide
- R1: renamed from R7; footprint (none) -> Resistors_ThroughHole:Resistor_Horizontal_RM10mm
- R10: renamed from R5; footprint (none) -> Resistors_ThroughHole:Resistor_Horizontal_RM10mm
- R11: renamed from R1; footprint (none) -> Resistors_ThroughHole:Resistor_Horizontal_RM10mm
- R2: renamed from R6; footprint (none) -> Resistors_ThroughHole:Resistor_Horizontal_RM10mm
- R3: renamed from R8; footprint (none) -> Resistors_ThroughHole:Resistor_Horizontal_RM10mm
- R4: renamed from R2; footprint (none) -> Resistors_ThroughHole:Resistor_Horizontal_RM10mm
- R5: renamed from R3; footprint (none) -> Resistors_ThroughHole:Resistor_Horizontal_RM10mm
- R6: renamed from R9; footprint (none) -> Resistors_ThroughHole:Resistor_Horizontal_RM10mm
- R7: renamed from R10; value 250 -> 270; footprint (none) -> Resistors_ThroughHole:Resistor_Horizontal_RM10mm
- R8: renamed from R11; value 410 -> 1k; footprint (none) -> Resistors_ThroughHole:Resistor_Horizontal_RM10mm
- R9: renamed from R4; footprint (none) -> Resistors_ThroughHole:Resistor_Horizontal_RM10mm
- U1: renamed from U2; footprint TO-220 -> TO_SOT_Packages_THT:TO-220_Neutral123_Horizontal
- U2: renamed from U1; footprint (none) -> Housings_DIP:DIP-8_W7.62mm
- Y1: footprint Crystals:Crystal_HC49-U_Vertical -> Crystals:Crystal_HC49-U_Horizontal_Typ2
- renumbered C4 to C1, P3 to P12, P7 to P3, P8 to P4, P1 to P6, P2 to P7
Connections:
- net labels added: MOT1F, MOT1PWM, MOT1R, MOT2F, MOT2PWM, MOT2R, USB1, USB2
- net labels removed: PUMP1, PUMP2
- wire segments 166 -> 216
- no-connect marks 21 -> 15
Other:
- moved on the sheet: C4, C5, C6, IC1, P1, P12, P2, P5, Q2, Q3, Q4, Q5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

Commit message: Finalized version 1.0
Parts:
- removed D2: 1N5818, symbol ZENER
- added C7: 10u, Capacitors_ThroughHole:C_Radial_D10_L20_P2.5, symbol CP1
- added D2: 1N5818, Diodes_ThroughHole:Diode_DO-35_SOD27_Horizontal_RM10, symbol D_Schottky
- added P14: ANALOG_IN, Pin_Headers:Pin_Header_Straight_1x11, symbol CONN_01X11
- added P15: PWM_IO, Pin_Headers:Pin_Header_Straight_1x04, symbol CONN_01X04
- added R12, R13: 10k, Resistors_ThroughHole:Resistor_Horizontal_RM10mm, symbol R
- added SW2: ISP_SELECT_JP, Pin_Headers:Pin_Header_Straight_1x03, symbol SWITCH_INV
- C1: footprint (none) -> Capacitors_ThroughHole:C_Radial_D10_L13_P5
- D1: footprint (none) -> Diodes_ThroughHole:Diode_DO-35_SOD27_Horizontal_RM10
- L1: footprint (none) -> Choke_Toroid_ThroughHole:Choke_Toroid_5x10mm_Vertical
- P1: value WATER_PUMP -> MOT2
- P2: value SPRAY_PUMP -> MOT1
- P3: value WATER_TANK -> INT0
- P4: value POT_BASE -> INT1
- U1: footprint TO_SOT_Packages_THT:TO-220_Neutral123_Horizontal -> TO_SOT_Packages_THT:TO-220_Neutral123_Vertical
- Y1: footprint Crystals:Crystal_HC49-U_Horizontal_Typ2 -> Crystals:Crystal_HC49-U_Vertical
Connections:
- net labels added: /SS
- wire segments 216 -> 251
- no-connect marks 15 -> 6
Other:
- moved on the sheet: C1, C2, C3, D1, L1, P10, P11, P12, P7, P8, P9, U2
